File: untitled.brd (EAGLE design)
At the start: 76.2 x 31.4 mm, 45 parts, among them IC1 NINA-B306-00B, IC2 INA126E, IC3 MCP6001T_SOT23, IC4 MAX8559ETAAA+T, J1 CSP-USC16-TR, J2 1761681-7, Q1 NTR5103NT1G, Q2 NTR5103NT1G, T1+ TESTPOINT_TPS-SMD-10SN, T1- TESTPOINT_TPS-SMD-10SN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

Commit message: Reset arrange insert
Parts:
- added C13: 0.1 uF, rcl:C0603
- added S1: BUTT-2, BUTT-2:SW_BUTT-2
Connections:
- new net RESET: C13.1, S1.1
- net GND: now also C13.2, S1.2
Changed lines of the file:
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@@
 <attribute name="VALUE" x="66.04" y="10.16" size="1.27" layer="27" align="center"/>
+</element>
+<element name="S1" library="BUTT-2" package="SW_BUTT-2" value="BUTT-2" x="-17.78" y="-1.27" smashed="yes">
+<attribute name="AVAILABILITY" value="In Stock" x="-17.78" y="-1.27" size="1.778" layer="27" display="off"/>
+<attribute name="DESCRIPTION" value=" Tactile Switches MINI PUSH BUTTON SWITCH 2-PIN QTY. 4 " x="-17.78" y="-1.27" size="1.778" layer="27" display="off"/>
+<attribute name="MF" value="Gravitech" x="-17.78" y="-1.27" size="1.778" layer="27" display="off"/>
+<attribute name="MP" value="BUTT-2" x="-17.78" y="-1.27" size="1.778" layer="27" display="off"/>
+<attribute name="NAME" x="-20.78" y="2.23" size="1.27" layer="25"/>
+<attribute name="PACKAGE" value="None" x="-17.78" y="-1.27" size="1.778" layer="27" display="off"/>
+<attribute name="PRICE" value="None" x="-17.78" y="-1.27" size="1.778" layer="27" display="off"/>
+<attribute name="PURCHASE-URL" value="https://pricing.snapeda.com/search/part/BUTT-2/?ref=eda" x="-17.78" y="-1.27" size="1.778" layer="27" display="off"/>
+<attribute name="VALUE" x="-20.78" y="-4.77" size="1.27" layer="27" align="top-left"/>
+</element>
+<element name="C13" library="rcl" library_urn="urn:adsk.eagle:library:334" package="C0603" package3d_urn="urn:adsk.eagle:package:23616/2" value="0.1 uF" x="-19.05" y="-11.43" smashed="yes">
+<attribute name="NAME" x="-19.685" y="-10.795" size="1.27" layer="25"/>
+<attribute name="POPULARITY" value="73" x="-19.05" y="-11.43" size="1.778" layer="27" display="off"/>
+<attribute name="SPICEPREFIX" value="C" x="-19.05" y="-11.43" size="1.778" layer="27" display="off"/>
+<attribute name="VALUE" x="-19.685" y="-13.335" size="1.27" layer="27"/>
 </element>
 </elements>
@@
 <contactref element="U$1" pad="4"/>
 <contactref element="GNDT1" pad="TP"/>
+<contactref element="S1" pad="2"/>
+<contactref element="C13" pad="2"/>
 <wire x1="42.205" y1="18.1928" x2="49.825" y2="18.1928" width="0" layer="19" extent="1-1"/>
 <wire x1="34.585" y1="18.1928" x2="42.205" y2="18.1928" width="0" layer="19" extent="1-1"/>
@@
 <wire x1="13.97" y1="23.71" x2="15.24" y2="25.82" width="0" layer="19" extent="1-1"/>
 <wire x1="2.81" y1="22.34" x2="2.54" y2="27.52" width="0" layer="19" extent="1-1"/>
+<wire x1="-15.28" y1="-1.27" x2="2.85" y2="7.105" width="0" layer="19" extent="1-1"/>
+<wire x1="-18.2" y1="-11.43" x2="-15.28" y2="-1.27" width="0" layer="19" extent="1-1"/>
 </signal>
 <signal name="N$1">
@@
 <contactref element="U$1" pad="1"/>
 </signal>
+<signal name="RESET">
+<contactref element="C13" pad="1"/>
+<contactref element="S1" pad="1"/>
+<wire x1="-20.28" y1="-1.27" x2="-19.9" y2="-11.43" width="0" layer="19" extent="1-1"/>
+</signal>
 </signals>
 <mfgpreviewcolors>
@@
 </drawing>
 <compatibility>
+<note version="6.3" minversion="6.2.2" severity="warning">
+Since Version 6.2.2 text objects can contain more than one line,
+which will not be processed correctly with this version.
+</note>
 <note version="8.2" severity="warning">
 Since Version 8.2, EAGLE supports online libraries. The ids

Commit message: first edit
Parts:
- added J3: DM3CS-SF-PEJMS, DM3CS-SF-PEJMS:DM3CSSFPEJMS
- moved C13 98.8 mm to (68.6, 34.3)
- moved S1 97.1 mm to (68.6, 43.2)
- moved R8 62.5 mm to (64.8, -11.4), turned to 270 degrees
- moved C11 61.5 mm to (61.0, -11.4)
- moved C10 60.5 mm to (57.1, -11.4)
- moved C5 59.5 mm to (53.3, -11.4)
- moved C4 58.5 mm to (49.5, -11.4)
- moved C3 57.6 mm to (45.7, -11.4)
- moved U2 24.4 mm to (20.3, 34.3), turned to 180 degrees
- moved U$1 23.0 mm to (68.6, 6.35), turned to 180 degrees
- moved J2 20.5 mm to (49.5, 47.0)
- moved U1 19.4 mm to (31.8, 34.3), turned to 180 degrees
- moved U4 19.4 mm to (54.6, 34.3), turned to 180 degrees
- moved U3 19.0 mm to (43.2, 34.3), turned to 180 degrees
- moved IC1 15.3 mm to (67.3, 25.4)
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Other:
- board size 76.2 x 31.4 mm -> 76.2 x 50.8 mm
