File: untitled.sch (EAGLE design)
At the start: 45 parts, among them IC1 NINA-B306-00B, IC2 INA126E, IC3 MCP6001T_SOT23, IC4 MAX8559ETAAA+T, J1 CSP-USC16-TR, J2 1761681-7, Q1 NTR5103NT1G, Q2 NTR5103NT1G, T1+ TESTPOINT_TPS-SMD-10SN, T1- TESTPOINT_TPS-SMD-10SN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

Commit message: Reset arrange insert
Parts:
- added C13: 0.1 uF, rcl:C-EUC0603
- added S1: BUTT-2, BUTT-2:BUTT-2
Connections:
- new net RESET: C13.1, S1.1
- net GND: now also C13.2, S1.2
Changed lines of the file:
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@@
 <part name="GNDT1" library="52101-101-REV-A_v16" library_urn="urn:adsk.eagle:library:21899384" deviceset="TESTPOINT_TPS" device="-SMD-10SN" package3d_urn="urn:adsk.eagle:package:15662280/2"/>
 <part name="IC1" library="NINA-B306-00B" deviceset="NINA-B306-00B" device="" override_package3d_urn="urn:adsk.eagle:package:37871514/2" override_package_urn="urn:adsk.eagle:footprint:37871515/1"/>
+<part name="S1" library="BUTT-2" deviceset="BUTT-2" device=""/>
+<part name="C13" library="rcl" library_urn="urn:adsk.eagle:library:334" deviceset="C-EU" device="C0603" package3d_urn="urn:adsk.eagle:package:23616/2" value="0.1 uF"/>
+<part name="GND29" library="audio amplifier example" library_urn="urn:adsk.eagle:library:970892" deviceset="GND" device="" value="SUP"/>
+<part name="GND30" library="audio amplifier example" library_urn="urn:adsk.eagle:library:970892" deviceset="GND" device="" value="SUP"/>
 </parts>
 <sheets>
@@
 <attribute name="VALUE" x="433.07" y="81.28" size="1.778" layer="96" align="center-left"/>
 </instance>
+<instance part="S1" gate="G$1" x="396.24" y="-33.02" smashed="yes">
+<attribute name="NAME" x="391.16" y="-29.21" size="1.778" layer="95"/>
+<attribute name="VALUE" x="391.16" y="-36.83" size="1.778" layer="96"/>
+</instance>
+<instance part="C13" gate="G$1" x="383.54" y="-38.1" smashed="yes">
+<attribute name="NAME" x="385.064" y="-37.719" size="1.778" layer="95"/>
+<attribute name="VALUE" x="385.064" y="-42.799" size="1.778" layer="96"/>
+</instance>
+<instance part="GND29" gate="G$1" x="383.54" y="-43.18" smashed="yes"/>
+<instance part="GND30" gate="G$1" x="403.86" y="-35.56" smashed="yes"/>
 </instances>
 <busses>
@@
 <pinref part="U$1" gate="A" pin="VSS"/>
 </segment>
+<segment>
+<pinref part="S1" gate="G$1" pin="2"/>
+<wire x1="403.86" y1="-33.02" x2="403.86" y2="-35.56" width="0.1524" layer="91"/>
+<pinref part="GND30" gate="G$1" pin="GND"/>
+</segment>
+<segment>
+<pinref part="C13" gate="G$1" pin="2"/>
+<pinref part="GND29" gate="G$1" pin="GND"/>
+</segment>
 </net>
 <net name="N$1" class="0">
@@
 </segment>
 </net>
+<net name="RESET" class="0">
+<segment>
+<pinref part="C13" gate="G$1" pin="1"/>
+<wire x1="383.54" y1="-35.56" x2="383.54" y2="-33.02" width="0.1524" layer="91"/>
+<pinref part="S1" gate="G$1" pin="1"/>
+<wire x1="383.54" y1="-33.02" x2="388.62" y2="-33.02" width="0.1524" layer="91"/>
+<label x="383.54" y="-33.02" size="1.27" layer="95" rot="R180" xref="yes"/>
+</segment>
+</net>
 </nets>
 </sheet>
@@
 </drawing>
 <compatibility>
+<note version="6.3" minversion="6.2.2" severity="warning">
+Since Version 6.2.2 text objects can contain more than one line,
+which will not be processed correctly with this version.
+</note>
 <note version="8.2" severity="warning">
 Since Version 8.2, EAGLE supports online libraries. The ids

Commit message: first edit
Parts:
- added J3: DM3CS-SF-PEJMS, DM3CS-SF-PEJMS:DM3CS-SF-PEJMS
Other:
- note added: "Front End"
- note added: "Headers & Reset"
- note added: "MUXes"
- note added: "Power Supply"
- note added: "USB C Interface"
- note added: "uController"
- moved on the sheet: 3V3T1, 5VMT1, C1, C10, C11, C12, C13, C2, C3, C4, C5, C6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
