File: untitled.sch (EAGLE design)
At the start: 48 parts, among them IC1 NINA-B306-00B, IC2 INA126E, IC3 MCP6001T_SOT23, IC4 MAX8559ETAAA+T, J1 USB4105-GF-A, J2 1761681-7, J3 DM3CS-SF-PEJMS, Q1 NTR5103NT1G, Q2 NTR5103NT1G, T1+ TESTPOINT_TPS-SMD-10SN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

Commit message: lista actualizada de pendientes
faltan algunas cosas, pero la base ya está para solo unir y rutear
Parts:
- removed T1+, T1-: TESTPOINT_TPS-SMD-10SN, 52101-101-REV-A_v16:TESTPOINT_TPS-SMD-10SN
- added FID1, FID4: FIDUCIAL_1MM, microbuilder:FIDUCIAL_1MM
- added J4: DNP, Arduino-connectors:PINHD-2X03(NO4)
- added R13: DNP, Arduino-rcl:R-DNP-0402
- added SJ1, SJ2: JUMPER-SMT_2_NO_NO-SILK, SparkFun-Jumpers:JUMPER-SMT_2_NO_NO-SILK
- added T1N, T1P: TESTPOINT_TPS-SMD-10SN, 52101-101-REV-A_v16:TESTPOINT_TPS-SMD-10SN
- added U$2, U$24, U$3, U$4: MOUNTINGHOLE2.5, microbuilder:MOUNTINGHOLE2.5
- renumbered U$1 to RV1
Connections:
- new net +3V3: J4.1, R13.1
- new net RESETN: J4.6
- new net SWCLK: J4.3, R13.2
- new net SWDIO: J4.2
- new net USB_N: SJ2.2
- new net USB_P: SJ1.2
- net GND: now also J4.5
- net USB+: now also SJ1.1, T1P.TP; no longer T1+.TP
- net USB-: now also SJ2.1, T1N.TP; no longer T1-.TP
Other:
- note added: "Añadir ADC ADS1220 (OPTIONAL)"
- note added: "Añadir conector plano de +42 pines (OPTIONAL)"
- note added: "Añadir headers para sacar i2c y spi"
- note added: "Añadir ic para carga y descarga de baterías?"
- note added: "Conectar MCU a pines"
- note added: "Controlar la salida 2 del regulador para encender/apagar circuitos"
- note added: "NTC MUX Board Rev1.4"
- note added: "SOLO VA UNO?"
- note added: "Sockets & Headers"
- note added: "TO DO LIST"
- note added: "Validar conexión spi y componentes para micro SD"
- note added: "Validar secuencia en MUXes"
- note removed: "Headers & Reset"
- moved on the sheet: 3V3T1, 5VMT1, C1, C10, C11, C13, C2, C3, C4, C5, C6, C7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
